Commit message: Added kinect, calibration not correct

File: cob_hardware_config/raw3-6/urdf/raw3-6.urdf.xacro (robot description, xacro)
@@ -11,4 +11,6 @@
   <!-- raw base -->
   <include filename="$(find raw_description)/urdf/base_long/base.urdf.xacro" />
+   <!--kinect-->
+ <include filename="$(find cob_description)/urdf/sensors/kinect.urdf.xacro" />
   <!-- raw tower -->
   <include filename="$(find raw_description)/urdf/tower_symetric/tower.urdf.xacro" />
@@ -19,3 +21,7 @@
       <origin xyz="${tower_x} ${tower_y} ${tower_z}" rpy="${tower_roll} ${tower_pitch} ${tower_yaw}" />
   </xacro:tower_symetric>
+  <!-- cam3d -->
+  <xacro:cob_kinect_v0 name="raw_cam3d" ros_topic="cam3d" parent="base_link">
+        <origin xyz=".51 0 .48" rpy="0 0 0" />
+  </xacro:cob_kinect_v0>
   </robot>
